File: hardware/kicad/ads1219.kicad_pcb (KiCad board)
At the start: 2 copper layers, 17.8 x 26.7 mm, 21 parts, among them J1 Conn_01x10, U1 ADS1219

Commit message: Add files via upload
Parts:
- J1: moved to B.Cu
- turned J1 to 180 degrees
